File: Hardware/Basic/Bottom/WatchX-BASIC-BOTTOM.brd (EAGLE design)
At the start: 33 x 33 mm, 31 parts, among them U1 AD5242-SO16

Commit message: changes up to take 003
Parts:
- added C1: 100n, LinnesLab-Passives:C0603
- added J1: (no value), LinnesLab-Connectors:1X07_1.27MM
- moved R19 35.0 mm to (33.5, 10.2), turned to 270 degrees
- moved R20 31.0 mm to (29.2, 6.97), turned to 180 degrees
- moved C15 29.5 mm to (29.2, 5.03), turned to 0 degrees
- moved R13 27.5 mm to (33.5, 6.79), turned to 270 degrees
- moved R21 27.1 mm to (31.9, 19.3), turned to 270 degrees
- moved R23 27.0 mm to (29.1, 25.2), turned to 180 degrees
- moved C19 24.6 mm to (29.1, 23.1), turned to 180 degrees
- moved R22 24.2 mm to (29.2, 21.1)
- moved IMU1 22.9 mm to (6.20, 28.6), turned to 90 degrees
- moved R16 22.9 mm to (18.8, 29.7)
- moved C14 20.6 mm to (29.2, 8.89), turned to 180 degrees
- moved C11 18.8 mm to (25.0, 10.0), turned to 90 degrees
- moved C20 18.6 mm to (21.3, 7.04), turned to 270 degrees
- moved U1 17.6 mm to (10.4, 9.75)
- moved R14 17.6 mm to (29.2, 10.9), turned to 0 degrees
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Connections:
- removed net LED: Q1.3
- removed net LED.CTRL: U$4.8
- removed net PPG: C21.2, OP3.1, U1.14
- removed net TIA: C10.2, C15.1, OP4.1, U1.3
- new net A6/TIA: C10.2, C15.1, J1.6, OP4.1, U1.3
- new net A7/PPG: C21.2, J1.7, OP3.1, U1.14
- new net D29/LED.CTRL: J1.5, U$4.8
- net 3.3V: now also J1.4
- net GND: now also C1.2, J1.3
- net LED.C: now also Q1.3
- net SCL: now also J1.2
- net SDA: now also J1.1
- net VREF: now also C1.1
Routing:
- net A6/TIA: track 0.00 -> 65.5 mm, vias 0 -> 4
- net A7/PPG: track 0.00 -> 64.3 mm, vias 0 -> 2
- net SCL: track 0.00 -> 52.0 mm, vias 0 -> 2
- net VREF: track 0.00 -> 37.2 mm, vias 0 -> 3
- net SDA: track 0.00 -> 34.7 mm
- net PD.C: track 0.00 -> 27.0 mm, vias 0 -> 2
- net GND: track 0.00 -> 25.5 mm, vias 0 -> 15
- net N$19: track 0.00 -> 24.4 mm
- net N$9: track 0.00 -> 18.9 mm
- net G.W2: track 0.00 -> 17.5 mm, vias 0 -> 2
- net N$13: track 0.00 -> 17.0 mm
- net D29/LED.CTRL: track 0.00 -> 15.4 mm, vias 0 -> 2
- net N$17: track 0.00 -> 10.4 mm, vias 0 -> 2
- net N$16: track 0.00 -> 10.3 mm
- net N$15: track 0.00 -> 7.72 mm
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- added copper zone on layer 16, net GND
